File: lcrmeter.sch (KiCad schematic (older format))
At the start: 35 parts, among them J1 inductor, J2 inductor, J3 gen, J4 1,5V, J5 gen, J6 OSC, J7 OSC, SW1 power, SW2 +, SW3 -, SW4 ok, SW5 back, U1 MCP47, U2 STM32F103C8Tx, Y1 8Mhz

Commit message: added most of new components
Parts:
- removed DIS1: nokia5110_LCD, Moje:LCD_5110, symbol lcrmeter-rescue:nokia5110_LCD
- removed J3: gen, Socket_Strips:Socket_Strip_Straight_1x02_Pitch2.54mm, symbol lcrmeter-rescue:Conn_01x02_Female
- removed J4: 1,5V, Socket_Strips:Socket_Strip_Straight_1x02_Pitch2.54mm, symbol lcrmeter-rescue:Conn_01x02_Female
- removed J5: gen, Pin_Headers:Pin_Header_Straight_1x02_Pitch2.54mm, symbol lcrmeter-rescue:Conn_01x02_Male
- removed L1: 10u, Inductors_SMD:L_0805_HandSoldering, symbol Device:L
- removed R2: 4K7, Resistors_SMD:R_0805_HandSoldering, symbol Device:R
- removed R3, R4, R5, R6: 10k, Resistors_SMD:R_0805_HandSoldering, symbol Device:R
- added C? (x5): 100n, symbol Device:C_Small
- added C?: 100n, Capacitors_SMD:C_0805_HandSoldering, symbol Device:C
- added C?: 10u, Capacitors_SMD:C_0805_HandSoldering, symbol Device:C
- added C?: 2u2, Capacitors_SMD:C_0805_HandSoldering, symbol Device:C
- added J?: Conn_01x04, symbol Connector_Generic:Conn_01x04
- added R? (x2): 10k, symbol Device:R_Small
- added R? (x8): 10k, Resistors_SMD:R_0805_HandSoldering, symbol Device:R
- added TP?: Reset, symbol Connector:TestPoint
- added U?: OLED, symbol Mylibrary:OLED
- added U? (x5): 74HC14, symbol 74xx:74HC14
- C7: value 10n -> 100n
- J1, J2: value inductor -> LCR_input
- R1: value R -> 100
Connections:
- net labels added: 8_MHz_OUT, ADC_1, ADC_2, BUTTON_+, BUTTON_-, BUTTON_BACK, BUTTON_OK, I2C_SCL, I2C_SDA, LATCH, OSCILLOSCOPE, PWM_OUT, SWO
- net labels removed: OSC
- wire segments 159 -> 145
- no-connect marks 0 -> 3
Other:
- note removed: "zmienić na kondensatory dorobić interfejs programistyczny\nrezystor 100 ohm- połączenie: dac-R-L-1,5V"

Commit message: schematic done
Parts:
- removed J6: OSC, Socket_Strips:Socket_Strip_Straight_1x02_Pitch2.54mm, symbol lcrmeter-rescue:Conn_01x02_Female
- removed J7: OSC, Pin_Headers:Pin_Header_Straight_1x02_Pitch2.54mm, symbol lcrmeter-rescue:Conn_01x02_Male
- removed J?: Conn_01x04, symbol Connector_Generic:Conn_01x04
- added D1, D2, D3, D4, D5, D6: BAT54S, Package_TO_SOT_SMD:SOT-23, symbol Diode:BAT54S
- added J3: Conn_01x06, symbol Connector_Generic:Conn_01x06
- added J4: USB_B_Micro, symbol Connector:USB_B_Micro
- added J5: OSCILLOSCOPE, symbol Connector:Conn_Coaxial
- added J6: misc, symbol Connector:Conn_01x06_Male
- added J7: misc, symbol Connector:Conn_01x06_Female
- added R14, R16: 22, symbol Device:R_Small
- added R15: 1k5, symbol Device:R_Small
- gave numbers to parts that had none: 21
Connections:
- net labels added: RST, USB_+, USB_-, USB_EN, VBUS
- wire segments 145 -> 162
- no-connect marks 3 -> 14
Other:
- note added: "Buttons"
- note added: "Caps"
- note added: "DAC"
- note added: "Power"
- note added: "TVS protection"
- note added: "miscellaneous\nconnectors"

Commit message: added voltage divider to oscilloscope
Parts:
- added R? (x2): 100, symbol Device:R
Connections:
- wire segments 162 -> 172
Changed lines of the file:
@@
 L Connector:Conn_Coaxial J5
 U 1 1 5C8FE9B7
-P 9425 6125
-F 0 "J5" H 9524 6101 50  0000 L CNN
-F 1 "OSCILLOSCOPE" H 9524 6010 50  0000 L CNN
-F 2 "" H 9425 6125 50  0001 C CNN
-F 3 " ~" H 9425 6125 50  0001 C CNN
-	1    9425 6125
+P 9505 5740
+F 0 "J5" H 9604 5716 50  0000 L CNN
+F 1 "OSCILLOSCOPE" H 9604 5625 50  0000 L CNN
+F 2 "" H 9505 5740 50  0001 C CNN
+F 3 " ~" H 9505 5740 50  0001 C CNN
+	1    9505 5740
 	1    0    0    -1
 $EndComp
@@
 L power:GND #PWR0135
 U 1 1 5C90A4C6
-P 9425 6325
-F 0 "#PWR0135" H 9425 6075 50  0001 C CNN
-F 1 "GND" H 9425 6175 50  0000 C CNN
-F 2 "" H 9425 6325 50  0001 C CNN
-F 3 "" H 9425 6325 50  0001 C CNN
-	1    9425 6325
-	1    0    0    -1
-$EndComp
-Text Label 9225 6125 2    50   ~ 0
+P 9560 6340
+F 0 "#PWR0135" H 9560 6090 50  0001 C CNN
+F 1 "GND" H 9560 6190 50  0000 C CNN
+F 2 "" H 9560 6340 50  0001 C CNN
+F 3 "" H 9560 6340 50  0001 C CNN
+	1    9560 6340
+	1    0    0    -1
+$EndComp
+Text Label 9230 6070 2    50   ~ 0
 OSCILLOSCOPE
 $Comp
@@
 	3665 4790 490  4790
 Wire Notes Line
-	11085 4625 8275 4625
-Wire Notes Line
-	3745 5125 8275 5125
-Wire Notes Line
-	8275 4625 8275 6555
-Wire Notes Line
 	8970 530  8970 2050
 Wire Notes Line
@@
 Wire Notes Line
 	1225 2030 1225 525
-Text Notes 7190 5510 0    100  ~ 0
+Text Notes 6795 5285 0    100  ~ 0
 Buttons
-Text Notes 8280 6490 0    100  ~ 0
+Text Notes 7690 6440 0    100  ~ 0
 miscellaneous\nconnectors
 Text Notes 9705 3590 1    100  ~ 0
@@
 Power
 NoConn ~ 9265 5510
+$Comp
+L Device:R R?
+U 1 1 5C873FB1
+P 9275 5910
+F 0 "R?" H 9345 5956 50  0000 L CNN
+F 1 "100" H 9345 5865 50  0000 L CNN
+F 2 "" V 9205 5910 50  0001 C CNN
+F 3 "~" H 9275 5910 50  0001 C CNN
+	1    9275 5910
+	1    0    0    -1
+$EndComp
+$Comp
+L Device:R R?
+U 1 1 5C874C9F
+P 9275 6235
+F 0 "R?" H 9345 6281 50  0000 L CNN
+F 1 "100" H 9345 6190 50  0000 L CNN
+F 2 "" V 9205 6235 50  0001 C CNN
+F 3 "~" H 9275 6235 50  0001 C CNN
+	1    9275 6235
+	1    0    0    -1
+$EndComp
+Wire Wire Line
+	9435 6385 9435 6340
+Wire Wire Line
+	9275 6385 9435 6385
+Wire Wire Line
+	9505 5940 9505 6340
+Wire Wire Line
+	9435 6340 9505 6340
+Connection ~ 9505 6340
+Wire Wire Line
+	9505 6340 9560 6340
+Wire Wire Line
+	9275 6085 9275 6070
+Wire Wire Line
+	9305 5740 9275 5740
+Wire Wire Line
+	9275 5740 9275 5760
+Wire Wire Line
+	9275 6070 9230 6070
+Connection ~ 9275 6070
+Wire Wire Line
+	9275 6070 9275 6060
+Wire Notes Line
+	11190 4715 7560 4715
+Wire Notes Line
+	7560 4715 7560 6505
+Wire Notes Line
+	7475 5110 3715 5110
 $EndSCHEMATC

Commit message: assigned footprints, fixed schematic, a little done PCB
Parts:
- removed D6: BAT54S, Package_TO_SOT_SMD:SOT-23, symbol Diode:BAT54S
- removed TP1: Reset, symbol Connector:TestPoint
- BT1, BT2: footprint Battery_Holders:Keystone_2466_1xAAA -> Battery:BatteryHolder_Keystone_2466_1xAAA
- C1, C11, C2: footprint Capacitors_SMD:C_0805_HandSoldering -> Capacitor_SMD:C_0805_2012Metric_Pad1.15x1.40mm_HandSolder
- C10, C12, C13, C14, C15: footprint (none) -> Capacitor_SMD:C_0603_1608Metric_Pad1.05x0.95mm_HandSolder
- C3, C4, C5, C6, C7, C8, C9: footprint Capacitors_SMD:C_0805_HandSoldering -> Capacitor_SMD:C_0603_1608Metric_Pad1.05x0.95mm_HandSolder
- J1: footprint Pin_Headers:Pin_Header_Straight_1x04_Pitch2.54mm -> Connector_PinHeader_2.54mm:PinHeader_1x04_P2.54mm_Vertical
- J2: footprint Socket_Strips:Socket_Strip_Straight_1x04_Pitch2.54mm -> Connector_PinSocket_2.54mm:PinSocket_1x04_P2.54mm_Vertical
- J3, J7: footprint (none) -> Connector_PinHeader_2.54mm:PinHeader_1x06_P2.54mm_Vertical
- J4: footprint (none) -> Connector_USB:USB_Micro-B_Molex_47346-0001
- J5: footprint (none) -> footprints:BNC TE CONNECTIVITY 5-1634503
- J6: footprint (none) -> Connector_PinSocket_2.54mm:PinSocket_1x06_P2.54mm_Vertical
- L2: footprint Inductors_SMD:L_0805_HandSoldering -> Inductor_SMD:L_0805_2012Metric_Pad1.15x1.40mm_HandSolder
- R1, R7, R8: footprint Resistors_SMD:R_0805_HandSoldering -> Resistor_SMD:R_0805_2012Metric_Pad1.15x1.40mm_HandSolder
- R10, R11, R12, R13, R4, R5, R6, R9: footprint Resistors_SMD:R_0805_HandSoldering -> Resistor_SMD:R_0603_1608Metric_Pad1.05x0.95mm_HandSolder
- R14, R15, R16: footprint (none) -> Resistor_SMD:R_0805_2012Metric_Pad1.15x1.40mm_HandSolder
- R17, R18: renamed from R?; footprint (none) -> Resistor_SMD:R_0805_2012Metric_Pad1.15x1.40mm_HandSolder
- R2, R3: footprint (none) -> Resistor_SMD:R_0603_1608Metric_Pad1.05x0.95mm_HandSolder
- SW1: footprint Pin_Headers:Pin_Header_Straight_1x03_Pitch2.54mm -> Connector_PinHeader_2.54mm:PinHeader_1x03_P2.54mm_Vertical
- SW2, SW3, SW4, SW5: footprint Buttons_Switches_SMD:SW_SPST_REED_CT05-XXXX-G1 -> Button_Switch_SMD:SW_SPST_REED_CT05-XXXX-G1
- U1: footprint Housings_SSOP:TSSOP-8_4.4x3mm_Pitch0.65mm -> Package_SO:TSSOP-8_4.4x3mm_P0.65mm
- U2: footprint Housings_QFP:LQFP-48_7x7mm_Pitch0.5mm -> Package_QFP:LQFP-48_7x7mm_P0.5mm
- U3: footprint (none) -> footprints:OLED_128x64
- U4: footprint (none) -> Package_SO:SOIC-14_3.9x8.7mm_P1.27mm
- Y1: footprint Crystals:Crystal_HC49-U_Vertical -> Crystal:Crystal_HC49-U_Vertical
Connections:
- wire segments 172 -> 171

Commit message: started routing added voltage divider for measuring supply foltage
Parts:
- added R19: 20k, Resistor_SMD:R_0805_2012Metric_Pad1.15x1.40mm_HandSolder, symbol Device:R
- added R20: 10k, Resistor_SMD:R_0805_2012Metric_Pad1.15x1.40mm_HandSolder, symbol Device:R
Connections:
- wire segments 171 -> 176
- no-connect marks 14 -> 13
Changed lines of the file:
@@
 NoConn ~ 2210 4320
 NoConn ~ 8010 3420
-NoConn ~ 8010 2920
 NoConn ~ 8010 2820
 Wire Notes Line
@@
 Wire Notes Line
 	7475 5110 3715 5110
+$Comp
+L Device:R R19
+U 1 1 5C8936BF
+P 8980 2735
+F 0 "R19" H 9050 2781 50  0000 L CNN
+F 1 "20k" H 9050 2690 50  0000 L CNN
+F 2 "Resistor_SMD:R_0805_2012Metric_Pad1.15x1.40mm_HandSolder" V 8910 2735 50  0001 C CNN
+F 3 "~" H 8980 2735 50  0001 C CNN
+	1    8980 2735
+	1    0    0    -1
+$EndComp
+$Comp
+L Device:R R20
+U 1 1 5C89377D
+P 8980 3090
+F 0 "R20" H 9050 3136 50  0000 L CNN
+F 1 "10k" H 9050 3045 50  0000 L CNN
+F 2 "Resistor_SMD:R_0805_2012Metric_Pad1.15x1.40mm_HandSolder" V 8910 3090 50  0001 C CNN
+F 3 "~" H 8980 3090 50  0001 C CNN
+	1    8980 3090
+	1    0    0    -1
+$EndComp
+Wire Wire Line
+	8980 2940 8980 2920
+Wire Wire Line
+	8010 2920 8980 2920
+Connection ~ 8980 2920
+Wire Wire Line
+	8980 2920 8980 2885
+$Comp
+L power:GND #PWR09
+U 1 1 5C8B821C
+P 8980 3270
+F 0 "#PWR09" H 8980 3020 50  0001 C CNN
+F 1 "GND" H 8980 3120 50  0000 C CNN
+F 2 "" H 8980 3270 50  0001 C CNN
+F 3 "" H 8980 3270 50  0001 C CNN
+	1    8980 3270
+	1    0    0    -1
+$EndComp
+Wire Wire Line
+	8980 3270 8980 3240
+$Comp
+L power:VCC #PWR08
+U 1 1 5C8BFA70
+P 8980 2550
+F 0 "#PWR08" H 8980 2400 50  0001 C CNN
+F 1 "VCC" H 8980 2700 50  0000 C CNN
+F 2 "" H 8980 2550 50  0001 C CNN
+F 3 "" H 8980 2550 50  0001 C CNN
+	1    8980 2550
+	1    0    0    -1
+$EndComp
+Wire Wire Line
+	8980 2550 8980 2585
 $EndSCHEMATC

Commit message: fixed resistors value, PCB done!
Parts:
- R17, R18: value 100 -> 10k; footprint Resistor_SMD:R_0805_2012Metric_Pad1.15x1.40mm_HandSolder -> Resistor_SMD:R_0603_1608Metric_Pad1.05x0.95mm_HandSolder
- R20: footprint Resistor_SMD:R_0805_2012Metric_Pad1.15x1.40mm_HandSolder -> Resistor_SMD:R_0603_1608Metric_Pad1.05x0.95mm_HandSolder
Changed lines of the file:
@@
 P 9275 5910
 F 0 "R17" H 9345 5956 50  0000 L CNN
-F 1 "100" H 9345 5865 50  0000 L CNN
-F 2 "Resistor_SMD:R_0805_2012Metric_Pad1.15x1.40mm_HandSolder" V 9205 5910 50  0001 C CNN
+F 1 "10k" H 9345 5865 50  0000 L CNN
+F 2 "Resistor_SMD:R_0603_1608Metric_Pad1.05x0.95mm_HandSolder" V 9205 5910 50  0001 C CNN
 F 3 "~" H 9275 5910 50  0001 C CNN
 	1    9275 5910
@@
 P 9275 6235
 F 0 "R18" H 9345 6281 50  0000 L CNN
-F 1 "100" H 9345 6190 50  0000 L CNN
-F 2 "Resistor_SMD:R_0805_2012Metric_Pad1.15x1.40mm_HandSolder" V 9205 6235 50  0001 C CNN
+F 1 "10k" H 9345 6190 50  0000 L CNN
+F 2 "Resistor_SMD:R_0603_1608Metric_Pad1.05x0.95mm_HandSolder" V 9205 6235 50  0001 C CNN
 F 3 "~" H 9275 6235 50  0001 C CNN
 	1    9275 6235
@@
 F 0 "R20" H 9050 3136 50  0000 L CNN
 F 1 "10k" H 9050 3045 50  0000 L CNN
-F 2 "Resistor_SMD:R_0805_2012Metric_Pad1.15x1.40mm_HandSolder" V 8910 3090 50  0001 C CNN
+F 2 "Resistor_SMD:R_0603_1608Metric_Pad1.05x0.95mm_HandSolder" V 8910 3090 50  0001 C CNN
 F 3 "~" H 8980 3090 50  0001 C CNN
 	1    8980 3090

Commit message: deleted 1,5V diode protection, added op-amp for 1,5V(optional), added zones
Parts:
- removed D1: BAT54S, Package_TO_SOT_SMD:SOT-23, symbol Diode:BAT54S
- added R21: 0, Resistor_SMD:R_2010_5025Metric_Pad1.52x2.65mm_HandSolder, symbol Device:R
- added R22, R23: 10k, Resistor_SMD:R_0603_1608Metric_Pad1.05x0.95mm_HandSolder, symbol Device:R
- added U5: MCP6001-OT, Package_TO_SOT_SMD:SOT-23-5, symbol Amplifier_Operational:MCP6001-OT
Connections:
- wire segments 176 -> 188
Other:
- note added: "Optional"
Changed lines of the file:
@@
 L power:+1V5 #PWR06
 U 1 1 5A1343EE
-P 970 1145
-F 0 "#PWR06" H 970 995 50  0001 C CNN
-F 1 "+1V5" H 970 1285 50  0000 C CNN
-F 2 "" H 970 1145 50  0001 C CNN
-F 3 "" H 970 1145 50  0001 C CNN
-	1    970  1145
+P 955 975
+F 0 "#PWR06" H 955 825 50  0001 C CNN
+F 1 "+1V5" H 955 1115 50  0000 C CNN
+F 2 "" H 955 975 50  0001 C CNN
+F 3 "" H 955 975 50  0001 C CNN
+	1    955  975
 	1    0    0    -1
 $EndComp
@@
 Wire Wire Line
 	610  770  610  725
-Wire Wire Line
-	585  1345 585  1360
-Wire Wire Line
-	970  1145 970  1360
-Wire Wire Line
-	970  1360 585  1360
-Connection ~ 585  1360
-Wire Wire Line
-	585  1360 585  1385
 $Comp
 L Device:R_Small R2
@@
 8_MHz_OUT
 $Comp
-L power:+1V5 #PWR0119
-U 1 1 5C861FBA
-P 9650 1380
-F 0 "#PWR0119" H 9650 1230 50  0001 C CNN
-F 1 "+1V5" H 9650 1520 50  0000 C CNN
-F 2 "" H 9650 1380 50  0001 C CNN
-F 3 "" H 9650 1380 50  0001 C CNN
-	1    9650 1380
-	1    0    0    -1
-$EndComp
-$Comp
-L power:VCC #PWR0120
-U 1 1 5C8623A1
-P 9400 1115
-F 0 "#PWR0120" H 9400 965 50  0001 C CNN
-F 1 "VCC" H 9400 1265 50  0000 C CNN
-F 2 "" H 9400 1115 50  0001 C CNN
-F 3 "" H 9400 1115 50  0001 C CNN
-	1    9400 1115
-	1    0    0    -1
-$EndComp
-$Comp
-L power:GND #PWR0121
-U 1 1 5C862650
-P 9400 1715
-F 0 "#PWR0121" H 9400 1465 50  0001 C CNN
-F 1 "GND" H 9400 1565 50  0000 C CNN
-F 2 "" H 9400 1715 50  0001 C CNN
-F 3 "" H 9400 1715 50  0001 C CNN
-	1    9400 1715
-	1    0    0    -1
-$EndComp
-$Comp
 L Connector_Generic:Conn_01x06 J3
 U 1 1 5C862939
@@
 	1    0    0    -1
 $EndComp
-$Comp
-L Diode:BAT54S D1
-U 1 1 5C8BDC1A
-P 9400 1415
-F 0 "D1" H 9400 1640 50  0000 C CNN
-F 1 "BAT54S" H 9400 1549 50  0000 C CNN
-F 2 "Package_TO_SOT_SMD:SOT-23" H 9475 1540 50  0001 L CNN
-F 3 "https://www.diodes.com/assets/Datasheets/ds11005.pdf" H 9280 1415 50  0001 C CNN
-	1    9400 1415
-	0    -1   -1   0
-$EndComp
-Wire Wire Line
-	9600 1415 9650 1415
-Wire Wire Line
-	9650 1415 9650 1380
 $Comp
 L Connector:Conn_01x06_Female J7
@@
 	3665 4790 490  4790
 Wire Notes Line
-	8970 530  8970 2050
-Wire Notes Line
-	8970 2050 9455 2050
-Wire Notes Line
 	9455 2050 9455 4625
 Wire Notes Line
@@
 Wire Wire Line
 	8980 2550 8980 2585
+$Comp
+L Amplifier_Operational:MCP6001-OT U5
+U 1 1 5C8BED48
+P 9140 1185
+F 0 "U5" H 9295 1295 50  0000 L CNN
+F 1 "MCP6001-OT" H 9125 1395 50  0000 L CNN
+F 2 "Package_TO_SOT_SMD:SOT-23-5" H 9040 985 50  0001 L CNN
+F 3 "http://ww1.microchip.com/downloads/en/DeviceDoc/21733j.pdf" H 9140 1385 50  0001 C CNN
+	1    9140 1185
+	1    0    0    -1
+$EndComp
+Wire Wire Line
+	585  1345 585  1355
+$Comp
+L Device:R R21
+U 1 1 5C8BFB53
+P 955 1150
+F 0 "R21" H 1025 1196 50  0000 L CNN
+F 1 "0" H 1025 1105 50  0000 L CNN
+F 2 "Resistor_SMD:R_2010_5025Metric_Pad1.52x2.65mm_HandSolder" V 885 1150 50  0001 C CNN
+F 3 "~" H 955 1150 50  0001 C CNN
+	1    955  1150
+	1    0    0    -1
+$EndComp
+Wire Wire Line
+	955  1000 955  975
+Wire Wire Line
+	955  1300 955  1355
+Wire Wire Line
+	955  1355 585  1355
+Connection ~ 585  1355
+Wire Wire Line
+	585  1355 585  1385
+Text Notes 1210 1300 1    50   ~ 0
+Optional
+$Comp
+L power:VCC #PWR018
+U 1 1 5C8CFAF1
+P 8595 675
+F 0 "#PWR018" H 8595 525 50  0001 C CNN
+F 1 "VCC" H 8595 825 50  0000 C CNN
+F 2 "" H 8595 675 50  0001 C CNN
+F 3 "" H 8595 675 50  0001 C CNN
+	1    8595 675
+	1    0    0    -1
+$EndComp
+$Comp
+L power:GND #PWR019
+U 1 1 5C8CFB7E
+P 8595 1590
+F 0 "#PWR019" H 8595 1340 50  0001 C CNN
+F 1 "GND" H 8595 1440 50  0000 C CNN
+F 2 "" H 8595 1590 50  0001 C CNN
+F 3 "" H 8595 1590 50  0001 C CNN
+	1    8595 1590
+	1    0    0    -1
+$EndComp
+$Comp
+L Device:R R22
+U 1 1 5C8CFF17
+P 8595 845
+F 0 "R22" H 8665 891 50  0000 L CNN
+F 1 "10k" H 8665 800 50  0000 L CNN
+F 2 "Resistor_SMD:R_0603_1608Metric_Pad1.05x0.95mm_HandSolder" V 8525 845 50  0001 C CNN
+F 3 "~" H 8595 845 50  0001 C CNN
+	1    8595 845
+	1    0    0    -1
+$EndComp
+$Comp
+L Device:R R23
+U 1 1 5C8D0B85
+P 8595 1300
+F 0 "R23" H 8665 1346 50  0000 L CNN
+F 1 "10k" H 8665 1255 50  0000 L CNN
+F 2 "Resistor_SMD:R_0603_1608Metric_Pad1.05x0.95mm_HandSolder" V 8525 1300 50  0001 C CNN
+F 3 "~" H 8595 1300 50  0001 C CNN
+	1    8595 1300
+	1    0    0    -1
+$EndComp
+Wire Wire Line
+	8840 1285 8840 1585
+Wire Wire Line
+	8840 1585 9440 1585
+Wire Wire Line
+	9440 1585 9440 1185
+Wire Wire Line
+	8595 1150 8595 1085
+Wire Wire Line
+	8595 1085 8840 1085
+Wire Wire Line
+	8595 995  8595 1085
+Connection ~ 8595 1085
+Wire Wire Line
+	8595 675  8595 695
+$Comp
+L power:VCC #PWR020
+U 1 1 5C8F08F3
+P 9040 860
+F 0 "#PWR020" H 9040 710 50  0001 C CNN
+F 1 "VCC" H 9040 1010 50  0000 C CNN
+F 2 "" H 9040 860 50  0001 C CNN
+F 3 "" H 9040 860 50  0001 C CNN
+	1    9040 860
+	1    0    0    -1
+$EndComp
+Wire Wire Line
+	9040 860  9040 885
+Wire Wire Line
+	8595 1450 8595 1485
+Connection ~ 8595 1485
+Wire Wire Line
+	8595 1485 8595 1590
+Wire Wire Line
+	8595 1485 9040 1485
+Wire Notes Line
+	10020 2050 10020 490
+$Comp
+L power:+1V5 #PWR021
+U 1 1 5C91B336
+P 9780 1120
+F 0 "#PWR021" H 9780 970 50  0001 C CNN
+F 1 "+1V5" H 9780 1260 50  0000 C CNN
+F 2 "" H 9780 1120 50  0001 C CNN
+F 3 "" H 9780 1120 50  0001 C CNN
+	1    9780 1120
+	1    0    0    -1
+$EndComp
+Wire Wire Line
+	9780 1120 9780 1185
+Wire Wire Line
+	9780 1185 9440 1185
+Connection ~ 9440 1185
+Wire Notes Line
+	8000 2050 8000 480
+Wire Notes Line
+	8000 2050 10020 2050
+Text Notes 9115 1820 0    50   ~ 0
+Optional
 $EndSCHEMATC

Commit message: fix oscilloscope connection
Connections:
- net labels added: OSCILLOSCOPE_IN
- wire segments 188 -> 192
Changed lines of the file:
@@
 $EndComp
 Text Label 10500 5025 2    50   ~ 0
-OSCILLOSCOPE
+OSCILLOSCOPE_IN
 $Comp
 L power:GND #PWR0109
@@
 8_MHz_OUT
 Text Label 10430 6005 0    50   ~ 0
-OSCILLOSCOPE
+OSCILLOSCOPE_IN
 $Comp
 L power:GND #PWR0132
@@
 L Connector:Conn_Coaxial J5
 U 1 1 5C8FE9B7
-P 9505 5740
-F 0 "J5" H 9604 5716 50  0000 L CNN
-F 1 "OSCILLOSCOPE" H 9604 5625 50  0000 L CNN
-F 2 "footprints:BNC TE CONNECTIVITY 5-1634503" H 9505 5740 50  0001 C CNN
-F 3 " ~" H 9505 5740 50  0001 C CNN
-	1    9505 5740
+P 8065 5195
+F 0 "J5" H 8164 5171 50  0000 L CNN
+F 1 "OSCILLOSCOPE" H 8164 5080 50  0000 L CNN
+F 2 "footprints:BNC TE CONNECTIVITY 5-1634503" H 8065 5195 50  0001 C CNN
+F 3 " ~" H 8065 5195 50  0001 C CNN
+	1    8065 5195
 	1    0    0    -1
 $EndComp
@@
 L power:GND #PWR0135
 U 1 1 5C90A4C6
-P 9560 6340
-F 0 "#PWR0135" H 9560 6090 50  0001 C CNN
-F 1 "GND" H 9560 6190 50  0000 C CNN
-F 2 "" H 9560 6340 50  0001 C CNN
-F 3 "" H 9560 6340 50  0001 C CNN
-	1    9560 6340
-	1    0    0    -1
-$EndComp
-Text Label 9230 6070 2    50   ~ 0
+P 8120 5795
+F 0 "#PWR0135" H 8120 5545 50  0001 C CNN
+F 1 "GND" H 8120 5645 50  0000 C CNN
+F 2 "" H 8120 5795 50  0001 C CNN
+F 3 "" H 8120 5795 50  0001 C CNN
+	1    8120 5795
+	1    0    0    -1
+$EndComp
+Text Label 7660 5510 3    50   ~ 0
 OSCILLOSCOPE
 $Comp
@@
 L Device:R R17
 U 1 1 5C873FB1
-P 9275 5910
-F 0 "R17" H 9345 5956 50  0000 L CNN
-F 1 "10k" H 9345 5865 50  0000 L CNN
-F 2 "Resistor_SMD:R_0603_1608Metric_Pad1.05x0.95mm_HandSolder" V 9205 5910 50  0001 C CNN
-F 3 "~" H 9275 5910 50  0001 C CNN
-	1    9275 5910
+P 7835 5365
+F 0 "R17" H 7905 5411 50  0000 L CNN
+F 1 "10k" H 7905 5320 50  0000 L CNN
+F 2 "Resistor_SMD:R_0603_1608Metric_Pad1.05x0.95mm_HandSolder" V 7765 5365 50  0001 C CNN
+F 3 "~" H 7835 5365 50  0001 C CNN
+	1    7835 5365
 	1    0    0    -1
 $EndComp
@@
 L Device:R R18
 U 1 1 5C874C9F
-P 9275 6235
-F 0 "R18" H 9345 6281 50  0000 L CNN
-F 1 "10k" H 9345 6190 50  0000 L CNN
-F 2 "Resistor_SMD:R_0603_1608Metric_Pad1.05x0.95mm_HandSolder" V 9205 6235 50  0001 C CNN
-F 3 "~" H 9275 6235 50  0001 C CNN
-	1    9275 6235
-	1    0    0    -1
-$EndComp
-Wire Wire Line
-	9435 6385 9435 6340
-Wire Wire Line
-	9275 6385 9435 6385
-Wire Wire Line
-	9505 5940 9505 6340
-Wire Wire Line
-	9435 6340 9505 6340
-Connection ~ 9505 6340
-Wire Wire Line
-	9505 6340 9560 6340
-Wire Wire Line
-	9275 6085 9275 6070
+P 7835 5690
+F 0 "R18" H 7905 5736 50  0000 L CNN
+F 1 "10k" H 7905 5645 50  0000 L CNN
+F 2 "Resistor_SMD:R_0603_1608Metric_Pad1.05x0.95mm_HandSolder" V 7765 5690 50  0001 C CNN
+F 3 "~" H 7835 5690 50  0001 C CNN
+	1    7835 5690
+	1    0    0    -1
+$EndComp
+Wire Wire Line
+	7995 5840 7995 5795
+Wire Wire Line
+	7835 5840 7995 5840
+Wire Wire Line
+	8065 5395 8065 5795
+Wire Wire Line
+	7995 5795 8065 5795
+Connection ~ 8065 5795
+Wire Wire Line
+	8065 5795 8120 5795
+Wire Wire Line
+	7835 5540 7835 5525
 Wire Wire Line
 	9305 5740 9275 5740
 Wire Wire Line
-	9275 5740 9275 5760
-Wire Wire Line
-	9275 6070 9230 6070
-Connection ~ 9275 6070
-Wire Wire Line
-	9275 6070 9275 6060
+	7835 5195 7835 5215
+Connection ~ 7835 5525
+Wire Wire Line
+	7835 5525 7835 5515
 Wire Notes Line
 	11190 4715 7560 4715
@@
 Text Notes 9115 1820 0    50   ~ 0
 Optional
+Wire Wire Line
+	7865 5195 7835 5195
+Wire Wire Line
+	7770 5525 7770 5510
+Wire Wire Line
+	7770 5510 7660 5510
+Wire Wire Line
+	7770 5525 7835 5525
+Text Label 7835 4975 0    50   ~ 0
+OSCILLOSCOPE_IN
+Wire Wire Line
+	7835 4975 7835 5195
+Connection ~ 7835 5195
 $EndSCHEMATC
